Commit message: finished joints section

File: body.urdf (robot description, URDF)
Before this commit: robot robot, 7 links, 6 joints
Links:
- removed link Link1
- removed link Link2
- removed link Link3
- removed link Link4
- removed link Link5
- removed link Link6
- removed link Link7
- added link Back_Leg, mass 1; collision box size=1 1 1; visual box size=1 1 1
- added link Body, mass 1; collision box size=1 1 1; visual box size=1 1 1
- added link Front_Leg, mass 1; collision box size=1 1 1; visual box size=1 1 1
Joints:
- removed joint Link1_Link2
- removed joint Link2_Link3
- removed joint Link3_Link4
- removed joint Link4_Link5
- removed joint Link5_Link6
- removed joint Link6_Link7
- added joint Back_Leg_Body: type revolute, parent Back_Leg, child Body, origin xyz=1 0 1 rpy=0 0 0, axis 0 1 0, limit lower=-3.14159 upper=3.14159 effort=0.0 velocity=0.0
- added joint Body_Front_Leg: type revolute, parent Body, child Front_Leg, origin xyz=1 0 0 rpy=0 0 0, axis 0 1 0, limit lower=-3.14159 upper=3.14159 effort=0.0 velocity=0.0

Commit message: finished sensors

File: body.urdf (robot description, URDF)
Before this commit: robot robot, 3 links, 2 joints
Links:
- removed link Back_Leg
- removed link Body
- removed link Front_Leg
- added link BackLeg, mass 1; collision box size=1 1 1; visual box size=1 1 1
- added link FrontLeg, mass 1; collision box size=1 1 1; visual box size=1 1 1
- added link Torso, mass 1; collision box size=1 1 1; visual box size=1 1 1
Joints:
- removed joint Back_Leg_Body
- removed joint Body_Front_Leg
- added joint Torso_BackLeg: type revolute, parent Torso, child BackLeg, origin xyz=1 0 1 rpy=0 0 0, axis 0 1 0, limit lower=-3.14159 upper=3.14159 effort=0.0 velocity=0.0
- added joint Torso_FrontLeg: type revolute, parent Torso, child FrontLeg, origin xyz=2 0 1 rpy=0 0 0, axis 0 1 0, limit lower=-3.14159 upper=3.14159 effort=0.0 velocity=0.0
